File: RegisterKicad/RegisterKicad.kicad_pcb (KiCad board)
At the start: 2 copper layers, 62.5 x 51.6 mm, 143 parts, among them J1 Conn_01x20_Pin, Q1 NPN, Q10 NPN, Q11 NPN, Q12 NPN, Q13 NPN, Q14 NPN, Q15 NPN, Q16 NPN, Q17 NPN, Q18 NPN, Q19 NPN, Q2 NPN, Q20 NPN, Q21 NPN, Q22 NPN, Q23 NPN, Q24 NPN, Q25 NPN, Q26 NPN, Q27 NPN, Q28 NPN, Q29 NPN, Q3 NPN, Q30 NPN, Q31 NPN, Q32 NPN, Q33 NPN, Q34 NPN, Q35 NPN, Q36 NPN, Q37 NPN, Q38 NPN, Q39 NPN, Q4 NPN, Q40 NPN, Q41 NPN, Q42 NPN, Q5 NPN, Q6 NPN, Q7 NPN, Q8 NPN, Q9 NPN

Commit message: feat: schematic and routed tri-state buffer pcb, also added "8-Bit Register" text to register pcb
Other:
- board text added: "8-Bit Register"
Changed lines of the file:
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@@
+		)
+	)
+	(gr_text "8-Bit Register"
+		(at 104.75 23.15 0)
+		(layer "F.SilkS")
+		(effects
+			(font
+				(size 3 3)
+				(thickness 0.6)
+				(bold yes)
+			)
+			(justify left bottom)
 		)
 	)

Commit message: feat: prod files for panelized tri-state buffer pcb. also bom update slightly
Parts:
- moved Q24 26.5 mm to (132.8, 66.3)
- moved Q9 26.5 mm to (143.5, 81.5)
- moved R47 26.5 mm to (131.8, 67.8)
- moved R8 26.5 mm to (142.4, 72.2)
- moved R83 26.5 mm to (135.7, 80.8)
- moved R49 26.5 mm to (136.7, 54.8)
- moved Q11 26.5 mm to (143.4, 92.3)
- moved Q12 26.5 mm to (150.5, 76.1)
- moved Q14 26.5 mm to (150.8, 87.0)
- moved Q15 26.5 mm to (150.7, 92.4)
- moved Q18 26.5 mm to (117.2, 70.5)
- moved Q2 26.5 mm to (108.1, 60.5)
- moved Q22 26.5 mm to (126.2, 70.7)
- moved Q23 26.5 mm to (132.8, 56.4)
- moved Q26 26.5 mm to (135.3, 70.3)
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Routing:
- net !WriteC: track 80.6 -> 81.3 mm
