File: TristateBufferKicad/TristateBufferKicad.kicad_pcb (KiCad board)
At the start: 2 copper layers, 66.5 x 48.5 mm, 60 parts, among them J1 Conn_01x19_Pin, Q1 NPN, Q10 NPN, Q11 NPN, Q12 NPN, Q13 NPN, Q14 NPN, Q15 NPN, Q16 NPN, Q17 NPN, Q18 NPN, Q19 NPN, Q2 NPN, Q20 NPN, Q21 NPN, Q22 NPN, Q23 NPN, Q24 NPN, Q25 NPN, Q3 NPN, Q4 NPN, Q5 NPN, Q6 NPN, Q7 NPN, Q8 NPN, Q9 NPN

Commit message: feat: prod files for panelized tri-state buffer pcb. also bom update slightly
Parts:
- moved Q10 0.07 mm to (149.5, 39.1)
- moved Q15 0.07 mm to (114.3, 58.8)
- moved Q18 0.07 mm to (129.1, 58.5)
- moved Q19 0.07 mm to (134.6, 53.8)
- moved Q20 0.07 mm to (141.0, 54.4)
- moved Q21 0.07 mm to (143.6, 58.5)
- moved Q22 0.07 mm to (149.1, 53.7)
- moved Q4 0.07 mm to (114.2, 43.8)
- moved Q8 0.07 mm to (141.4, 39.9)
- moved Q9 0.07 mm to (143.9, 43.9)
- moved R10 0.07 mm to (130.2, 41.5)
- moved R13 0.07 mm to (140.0, 45.5)
- moved R18 0.07 mm to (159.9, 42.0)
- moved R25 0.07 mm to (125.1, 60.3)
- moved R26 0.07 mm to (130.6, 56.4)
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Other:
- outline, holes or cut-outs redrawn
